File: pcb/3W6Uni/3W6Uni.kicad_pcb (KiCad board)
At the start: 2 copper layers, 236.8 x 106.5 mm, 95 parts, among them J1 USB_C Main, SW1 SW_Push, SW10 SW_Push, SW11 SW_Push, SW12 SW_Push, SW13 SW_Push, SW14 SW_Push, SW15 SW_Push, SW16 SW_Push, SW17 SW_Push, SW18 SW_Push, SW19 SW_Push, SW2 SW_Push, SW20 SW_Push, SW21 SW_Push, SW22 SW_Push, SW23 SW_Push, SW24 SW_Push, SW25 SW_Push, SW26 SW_Push, SW27 SW_Push, SW28 SW_Push, SW29 SW_Push, SW3 SW_Push, SW30 SW_Push, SW31 SW_Push, SW32 SW_Push, SW33 SW_Push, SW34 SW_Push, SW35 SW_Push, SW4 SW_Push, SW5 SW_Push, SW6 SW_Push, SW7 SW_Push, SW8 SW_Push, SW9 SW_Push, U1 ATmega32U4-AU, Y1 16MHZ

Commit message: add rotary encoder to lib.WIP PCB
Parts:
- added D35: D, Weteor:D_SOD-123, F.Cu at (149.1, 118.4)
- added SW36: Rotary_Encoder_Switch, Weteor:RotEncoderE11, B.Cu at (148.5, 106.1)
- C1, C2, C3, C4, C5, C6, C7, C8: footprint Weteor:C_0402_HandSolder -> Capacitor_SMD:C_0805_2012Metric_Pad1.18x1.45mm_HandSolder
- J1: moved to B.Cu
- R1, R2, R3, R4, R5, R6: footprint Weteor:R_0402_HandSolder -> Resistor_SMD:R_0805_2012Metric_Pad1.20x1.40mm_HandSolder
- moved D13 236.8 mm to (105.4, 113.9), turned to 339 degrees
- moved D6 231.0 mm to (65.2, 79.2), turned to 343 degrees
- moved D21 228.6 mm to (166.6, 126.9), turned to 36 degrees
- moved D12 218.2 mm to (99.8, 90.3), turned to 339 degrees
- moved D2 216.9 mm to (45.9, 68.8), turned to 354.5 degrees
- moved D19 179.3 mm to (174.3, 80.9), turned to 21 degrees
- moved R1 175.4 mm to (139.6, 73.0), turned to 90 degrees
- moved C2 175.2 mm to (136.9, 73.1), turned to 90 degrees
- moved D23 174.6 mm to (191.2, 74.5), turned to 21 degrees
- moved D8 171.4 mm to (90.5, 64.2), turned to 339 degrees
- moved D3 167.4 mm to (44.2, 85.8), turned to 354.5 degrees
- moved D20 162.7 mm to (180.4, 96.8), turned to 21 degrees
- moved D15 160.7 mm to (122.8, 80.9), turned to 339 degrees
- moved SW4 158.9 mm to (148.6, 133.3), turned to 180 degrees
- moved C3 155.1 mm to (143.5, 88.1), turned to 90 degrees
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Connections:
- U1 pad 10: /Row_2 -> Net-(U1-Pad10)
- U1 pad 11: /Row_3 -> Net-(U1-Pad11)
- U1 pad 12: /Col_3 -> Net-(U1-Pad12)
- U1 pad 20: /Col_6 -> /Col_4
- U1 pad 21: /Col_7 -> /Col_3
- U1 pad 22: /Col_9 -> /Col_2
- U1 pad 25: /Col_8 -> /Col_1
- U1 pad 26: Net-(U1-Pad26) -> /Col_0
- U1 pad 27: Net-(U1-Pad27) -> /Row_3
- U1 pad 28: /Col_0 -> /encA
- U1 pad 29: /Col_1 -> /encB
- U1 pad 30: /Col_2 -> /Col_9
- U1 pad 31: /Col_4 -> /Col_8
- U1 pad 32: /Col_5 -> /Col_7
- U1 pad 37: Net-(U1-Pad37) -> /Col_6
- U1 pad 38: Net-(U1-Pad38) -> /Col_5
- U1 pad 39: Net-(U1-Pad39) -> /Row_2
- U1 pad 40: Net-(U1-Pad40) -> /Row_1
- U1 pad 41: Net-(U1-Pad41) -> /Row_0
- U1 pad 8: /Row_0 -> Net-(U1-Pad8)
- U1 pad 9: /Row_1 -> Net-(U1-Pad9)
Routing:
- net /Row_2: track 0.00 -> 265.7 mm, vias 0 -> 2
- net /Row_0: track 0.00 -> 252.4 mm, vias 0 -> 2
- net /Row_1: track 0.00 -> 242.6 mm, vias 0 -> 2
- net /Col_9: track 0.00 -> 167.1 mm, vias 0 -> 1
- net /Col_0: track 0.00 -> 155.3 mm
- net /Col_2: track 0.00 -> 153.7 mm, vias 0 -> 2
- net /Col_6: track 0.00 -> 150.7 mm
- net /Row_3: track 0.00 -> 149.6 mm
- net /Col_8: track 0.00 -> 148.7 mm
- net /Col_1: track 0.00 -> 140.6 mm
- net /Col_5: track 0.00 -> 135.5 mm
- net /Col_7: track 0.00 -> 134.7 mm
- net /Col_3: track 0.00 -> 131.7 mm
- net /Col_4: track 0.00 -> 114.8 mm
- net +5V: track 0.00 -> 76.9 mm, vias 0 -> 3
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- added copper zone on B.Cu, net GND
Other:
- outline, holes or cut-outs redrawn

Commit message: pcb routed
Parts:
- removed R4: 22R, Resistor_SMD:R_0805_2012Metric_Pad1.20x1.40mm_HandSolder
- removed the REF** at (126.1, 53.4)
- removed the REF** at (170.9, 53.4)
- removed the REF** at (236.9, 50.8)
- removed the REF** at (237.7, 98.4)
- removed the REF** at (170.1, 112.8)
- removed the REF** at (126.9, 112.8)
- removed the REF** at (59.4, 98.4)
- removed the REF** at (60.2, 50.8)
- removed Y1: 16MHZ, Crystal:Crystal_SMD_3225-4Pin_3.2x2.5mm
- added BT1: Battery_Cell, Weteor:JST GH 2Pin, F.Cu at (117.1, 57.4)
- added C10: 0.1uF, Capacitor_SMD:C_0805_2012Metric, F.Cu at (161.9, 72.4)
- added C11: 1nF, Capacitor_SMD:C_0805_2012Metric, F.Cu at (140.8, 52.5)
- added C9: 100nF, Capacitor_SMD:C_0805_2012Metric, F.Cu at (142.4, 67.9)
- added D36: D_Schottky_Small, Diode_SMD:D_SOD-323_HandSoldering, F.Cu at (164.7, 58.2)
- added D37: gween, Diode_SMD:D_0805_2012Metric, F.Cu at (161.7, 54.8)
- added D38: oragne, Diode_SMD:D_0805_2012Metric, F.Cu at (159.0, 54.8)
- added J2: BL_CONN, Weteor:JST Gh Molex PicoBlade 4Pin, F.Cu at (76.7, 106.0)
- added Q1: AO3401A, Package_TO_SOT_SMD:SOT-23, F.Cu at (137.3, 58.5)
- added R10: 100R, Resistor_SMD:R_0805_2012Metric_Pad1.20x1.40mm_HandSolder, F.Cu at (167.0, 54.7)
- added R12: 1k, Resistor_SMD:R_0805_2012Metric_Pad1.20x1.40mm_HandSolder, F.Cu at (164.0, 54.7)
- added R13: 1k, Resistor_SMD:R_0805_2012Metric_Pad1.20x1.40mm_HandSolder, F.Cu at (156.6, 54.7)
- added R14: 5k, Resistor_SMD:R_0805_2012Metric_Pad1.20x1.40mm_HandSolder, F.Cu at (150.9, 63.4)
- added R15: 100, Resistor_SMD:R_0805_2012Metric_Pad1.20x1.40mm_HandSolder, F.Cu at (161.9, 68.5)
- added R16: 1k, Resistor_SMD:R_0805_2012Metric_Pad1.20x1.40mm_HandSolder, F.Cu at (154.1, 71.4)
- added R7: 100k, Resistor_SMD:R_0805_2012Metric_Pad1.20x1.40mm_HandSolder, F.Cu at (150.9, 65.8)
- added R8: 2R2, Resistor_SMD:R_0805_2012Metric_Pad1.20x1.40mm_HandSolder, F.Cu at (164.7, 60.4)
- added REF**: MountingHole_2.2mm_M2_DIN965_Pad_TopOnly, MountingHole:MountingHole_2.2mm_M2_DIN965_Pad_TopOnly, F.Cu at (50.1, 42.3)
- added REF**: MountingHole_2.2mm_M2_DIN965_Pad_TopOnly, MountingHole:MountingHole_2.2mm_M2_DIN965_Pad_TopOnly, F.Cu at (126.1, 53.4)
- added REF**: MountingHole_2.2mm_M2_DIN965_Pad_TopOnly, MountingHole:MountingHole_2.2mm_M2_DIN965_Pad_TopOnly, F.Cu at (250.7, 104.4)
- added REF**: MountingHole_2.2mm_M2_DIN965_Pad_TopOnly, MountingHole:MountingHole_2.2mm_M2_DIN965_Pad_TopOnly, F.Cu at (46.4, 104.4)
- added REF**: MountingHole_2.2mm_M2_DIN965_Pad_TopOnly, MountingHole:MountingHole_2.2mm_M2_DIN965_Pad_TopOnly, F.Cu at (246.9, 42.3)
- added REF**: MountingHole_2.2mm_M2_DIN965_Pad_TopOnly, MountingHole:MountingHole_2.2mm_M2_DIN965_Pad_TopOnly, F.Cu at (170.9, 53.4)
- added REF**: MountingHole_2.2mm_M2_DIN965_Pad_TopOnly, MountingHole:MountingHole_2.2mm_M2_DIN965_Pad_TopOnly, F.Cu at (170.1, 107.1)
- added REF**: MountingHole_2.2mm_M2_DIN965_Pad_TopOnly, MountingHole:MountingHole_2.2mm_M2_DIN965_Pad_TopOnly, F.Cu at (127.0, 107.1)
- added SW37: SW_RESET, Weteor:Micro_Push_Button_3x6x2.5mm, F.Cu at (161.9, 50.7)
- added U2: TP4056, Weteor:TP4056_SOP-8-PP, F.Cu at (157.8, 63.4)
- added U3: XC6206PxxxMR-Regulator_Linear, Package_TO_SOT_SMD:SOT-23, F.Cu at (142.4, 71.4)
- added U4: DW01A, Package_TO_SOT_SMD:SOT-23-6, F.Cu at (157.9, 72.4)
- added U5: FS8205, Package_TO_SOT_SMD:SOT-23-6, F.Cu at (157.9, 68.5)
- added U6: USBLC6-2SC6, Package_TO_SOT_SMD:SOT-23-6, F.Cu at (148.5, 58.4)
- C1, C2: value 22pF -> 10uF; footprint Capacitor_SMD:C_0805_2012Metric_Pad1.18x1.45mm_HandSolder -> Capacitor_SMD:C_0805_2012Metric
- C3: value 0.1uF -> 10uF; footprint Capacitor_SMD:C_0805_2012Metric_Pad1.18x1.45mm_HandSolder -> Capacitor_SMD:C_0805_2012Metric
- C4, C5: value 0.1uF -> 4.7uF; footprint Capacitor_SMD:C_0805_2012Metric_Pad1.18x1.45mm_HandSolder -> Capacitor_SMD:C_0805_2012Metric
- C6: value 0.1uF -> 1uF; footprint Capacitor_SMD:C_0805_2012Metric_Pad1.18x1.45mm_HandSolder -> Capacitor_SMD:C_0805_2012Metric
- C7: value 4.7uF -> 10uF; footprint Capacitor_SMD:C_0805_2012Metric_Pad1.18x1.45mm_HandSolder -> Capacitor_SMD:C_0805_2012Metric
- C8: footprint Capacitor_SMD:C_0805_2012Metric_Pad1.18x1.45mm_HandSolder -> Capacitor_SMD:C_0805_2012Metric
- R1: value 10k -> 806k
- R2: value 10k -> 2M
- R3: value 22R -> 1M
- SW36: footprint Weteor:RotEncoderE11 -> Weteor:RotEncoderE11_SMD
- SW4: value SW_Push -> ON_OFF; footprint Weteor:Micro_Push_Button_3x6x2.5mm -> Weteor:switch_MSK-12C02_smd
- U1: value ATmega32U4-AU -> MS88SF2; footprint Package_QFP:TQFP-44_10x10mm_P0.8mm -> ms88sf2_oreore:MINEW_MS88SF2
- moved SW4 85.0 mm to (135.2, 49.3), turned to -90 degrees
- moved U1 66.9 mm to (148.5, 144.9), turned to 180 degrees
- moved R1 60.6 mm to (161.5, 129.6), turned to 180 degrees
- moved C2 50.0 mm to (135.7, 123.0), turned to 180 degrees
- moved C1 47.8 mm to (161.5, 123.0), turned to 0 degrees
- moved R2 45.7 mm to (161.5, 131.8), turned to 0 degrees
- moved C3 33.2 mm to (159.7, 59.2), turned to 180 degrees
- moved C7 21.1 mm to (163.7, 64.4), turned to 90 degrees
- moved D35 18.6 mm to (166.5, 124.9)
- moved R3 13.7 mm to (140.8, 49.0)
- moved C5 13.4 mm to (150.7, 71.4), turned to 90 degrees
- moved C6 13.3 mm to (145.8, 71.4), turned to 90 degrees
- moved D14 9.56 mm to (120.8, 70.2)
- moved D10 9.55 mm to (104.0, 63.8)
- moved C4 6.72 mm to (148.3, 71.4), turned to 90 degrees
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Connections:
- net Net-(J1-PadA6) renamed /dbus+
- C1 pad 1: Net-(C1-Pad1) -> +3V3
- C3 pad 1: GND -> /vbus
- C3 pad 2: +5V -> GND
- C4 pad 1: GND -> /vbat
- C4 pad 2: +5V -> GND
- C5 pad 1: GND -> /vbat
- C5 pad 2: +5V -> GND
- C6 pad 1: GND -> /vbat
- C6 pad 2: +5V -> GND
- C7 pad 1: GND -> /vbat
- C7 pad 2: +5V -> GND
- C8 pad 1: Net-(C8-Pad1) -> /regbat
- F1 pad 2: +5V -> /vbus
- J1 pad A7: Net-(J1-PadA7) -> /dbus-
- J1 pad A8: Net-(J1-PadA8) -> unconnected-(J1-PadA8)
- J1 pad B7: Net-(J1-PadA7) -> /dbus-
- J1 pad B8: Net-(J1-PadB8) -> unconnected-(J1-PadB8)
- J1 pad S1: Net-(J1-PadS1) -> Earth
- R1 pad 1: +5V -> /vbat
- R1 pad 2: Net-(R1-Pad2) -> /vsense
- R2 pad 1: GND -> /vsense
- R2 pad 2: Net-(R2-Pad2) -> GND
- R3 pad 1: /D- -> Earth
- R3 pad 2: Net-(J1-PadA7) -> GND
- SW4 pad 1: GND -> /regbat
- SW4 pad 2: Net-(R1-Pad2) -> Net-(Q1-Pad3)
- U1 pad 1: /Col_L1 -> GND
- U1 pad 10: Net-(U1-Pad10) -> /Row_2
- U1 pad 11: Net-(U1-Pad11) -> /Row_1
- U1 pad 12: Net-(U1-Pad12) -> /Row_0
- U1 pad 13: Net-(R1-Pad2) -> GND
- U1 pad 14: +5V -> +3V3
- U1 pad 15: GND -> Net-(C2-Pad1)
- U1 pad 16: Net-(C2-Pad1) -> /d-
- U1 pad 17: Net-(C1-Pad1) -> /d+
- U1 pad 18: /I2C_SCL_L -> /Col_3
- U1 pad 19: /I2C_SDA_L -> /Col_2
- U1 pad 2: +5V -> /Col_5
- U1 pad 20: /Col_4 -> /reset
- U1 pad 21: /Col_3 -> /Col_1
- U1 pad 22: /Col_2 -> /Col_0
- U1 pad 23: GND -> /Col_4
- U1 pad 24: +5V -> unconnected-(U1-Pad24)
- U1 pad 25: /Col_1 -> /swdio
- U1 pad 26: /Col_0 -> /swclk
- U1 pad 27: /Row_3 -> /encA
- U1 pad 28: /encA -> /encB
- U1 pad 3: /D- -> /Col_9
- U1 pad 4: /D+ -> /Col_8
- U1 pad 5: GND -> /Col_7
- U1 pad 6: Net-(C8-Pad1) -> /vsense
- U1 pad 7: +5V -> unconnected-(U1-Pad7)
- U1 pad 8: Net-(U1-Pad8) -> /Col_6
- U1 pad 9: Net-(U1-Pad9) -> /Row_3
Routing:
- net +3V3: track 0.00 -> 157.2 mm, vias 0 -> 6
- net /vbat: track 0.00 -> 145.7 mm, vias 0 -> 6
- net /reset: track 0.00 -> 92.9 mm, vias 0 -> 2
- net /d+: track 0.00 -> 87.8 mm
- net /d-: track 0.00 -> 87.6 mm
- net /swdio: track 0.00 -> 87.4 mm, vias 0 -> 1
- net /swclk: track 0.00 -> 84.8 mm, vias 0 -> 2
- net +5V: track 76.9 -> 0.00 mm, vias 3 -> 0
- net Net-(C2-Pad1): track 9.94 -> 79.1 mm, vias 0 -> 2
- net Net-(BT1-Pad2): track 0.00 -> 60.1 mm, vias 0 -> 4
- net /Row_0: track 252.4 -> 311.4 mm, vias 2 -> 4
- net /vbus: track 0.00 -> 58.9 mm, vias 0 -> 5
- net /Row_1: track 242.6 -> 289.4 mm
- net /Col_5: track 135.5 -> 101.6 mm, vias 0 -> 1
- net /Row_3: track 149.6 -> 118.8 mm, vias 0 -> 2
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- added copper zone on F.Cu, net GND
Other:
- outline, holes or cut-outs redrawn
- net class Default removed
- rule pad_to_mask_clearance: 0 -> 0.05

Commit message: make pcb ready for manufacturing, add backplate
Parts:
- added J3: Conn_01x04, Connector_PinHeader_1.27mm:PinHeader_1x04_P1.27mm_Vertical, B.Cu at (42.7, 81.8)
- added J4: Conn_01x04, Connector_PinHeader_1.27mm:PinHeader_1x04_P1.27mm_Vertical, B.Cu at (44.4, 64.9)
- added J5: Conn_01x04, Connector_PinHeader_1.27mm:PinHeader_1x04_P1.27mm_Vertical, B.Cu at (250.6, 82.2)
- added J6: Conn_01x04, Connector_PinHeader_1.27mm:PinHeader_1x04_P1.27mm_Vertical, B.Cu at (248.9, 65.2)
- BT1: footprint Weteor:JST GH 2Pin -> Weteor:Molex PicoBlade 2Pin smt tht
- J2: footprint Weteor:JST Gh Molex PicoBlade 4Pin -> Weteor:Molex PicoBlade 4Pin smt tht
- moved J2 6.25 mm to (82.5, 108.2), turned to -111 degrees
- moved BT1 5.63 mm to (113.7, 52.9)
Connections:
- net Net-(D1-Pad2) renamed /LT_sw
- net Net-(D2-Pad2) renamed /LM_sw
- net Net-(D3-Pad2) renamed /LB_sw
- net Net-(D32-Pad2) renamed /RT_sw
- net Net-(D33-Pad2) renamed /RM_sw
- net Net-(D34-Pad2) renamed /RB_sw
Routing:
- net /RB_sw: track 13.1 -> 37.8 mm, vias 0 -> 1
- net /LB_sw: track 13.1 -> 35.9 mm, vias 0 -> 1
- net /swdio: track 87.4 -> 70.6 mm
- net /swclk: track 84.8 -> 70.1 mm, vias 2 -> 1
- net +3V3: track 157.2 -> 147.5 mm
- net /Col_9: track 166.0 -> 172.5 mm
- net /Col_0: track 145.9 -> 152.3 mm
- net /RM_sw: track 13.1 -> 18.8 mm, vias 0 -> 1
- net /LM_sw: track 13.1 -> 18.5 mm, vias 0 -> 1
- net /vbat: track 145.7 -> 149.9 mm
- net Net-(BT1-Pad2): track 60.1 -> 64.1 mm
- net /LT_sw: track 13.1 -> 16.9 mm
- net /RT_sw: track 13.1 -> 16.5 mm
- net /Row_2: track 287.9 -> 289.2 mm
- net GND: track 45.0 -> 43.9 mm, vias 29 -> 28
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Other:
- board text added: "Off"
- board text added: "On"
- board text added: "Reset"
