File: pcb/3W6Uni/3W6Uni.kicad_sch (KiCad schematic)
At the start: 110 parts, among them J1 USB_C Main, J2 BL_CONN, Q1 AO3401A, SW1 SW_Push, SW10 SW_Push, SW11 SW_Push, SW12 SW_Push, SW13 SW_Push, SW14 SW_Push, SW15 SW_Push, SW16 SW_Push, SW17 SW_Push, SW18 SW_Push, SW19 SW_Push, SW2 SW_Push, SW20 SW_Push, SW21 SW_Push, SW22 SW_Push, SW23 SW_Push, SW24 SW_Push, SW25 SW_Push, SW26 SW_Push, SW27 SW_Push, SW28 SW_Push, SW29 SW_Push, SW3 SW_Push, SW30 SW_Push, SW31 SW_Push, SW32 SW_Push, SW33 SW_Push, SW34 SW_Push, SW35 SW_Push, SW36 Rotary_Encoder_Switch, SW37 SW_RESET, SW4 ON_OFF, SW5 SW_Push, SW6 SW_Push, SW7 SW_Push, SW8 SW_Push, SW9 SW_Push, U1 MS88SF2, U2 TP4056, U3 XC6206PxxxMR-Regulator_Linear, U4 DW01A, U5 FS8205, U6 USBLC6-2SC6

Commit message: make pcb ready for manufacturing, add backplate
Parts:
- added J3, J4, J5, J6: Conn_01x04, Connector_PinHeader_1.27mm:PinHeader_1x04_P1.27mm_Vertical, symbol Connector_Generic:Conn_01x04
- BT1: footprint Weteor:JST GH 2Pin -> Weteor:Molex PicoBlade 2Pin smt tht
- J2: footprint Weteor:JST Gh Molex PicoBlade 4Pin -> Weteor:Molex PicoBlade 4Pin smt tht
Connections:
- net Col_0: now also J4.4 (Pin_4)
- net Col_9: now also J6.4 (Pin_4)
- net LT_sw: now reaches D1.2 (A), SW1.2
- net LT_sw: now also J4.1 (Pin_1)
- net LM_sw: now reaches D2.2 (A), SW2.2
- net LM_sw: now also J4.2 (Pin_2)
- net LB_sw: now reaches D3.2 (A), SW3.2
- net LB_sw: now also J4.3 (Pin_3)
- net RT_sw: now reaches D32.2 (A), SW33.2
- net RT_sw: now also J6.1 (Pin_1)
- net RM_sw: now reaches D33.2 (A), SW34.2
- net RM_sw: now also J6.2 (Pin_2)
- net RB_sw: now reaches D34.2 (A), SW35.2
- net RB_sw: now also J6.3 (Pin_3)
- no-connect marks 7 -> 15
Changed lines of the file:
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@@
   (junction (at 278.13 118.11) (diameter 1.016) (color 0 0 0 0))
   (junction (at 278.13 122.555) (diameter 1.016) (color 0 0 0 0))
+  (no_connect (at 27.94 107.95))
+  (no_connect (at 27.94 110.49))
+  (no_connect (at 27.94 113.03))
+  (no_connect (at 27.94 115.57))
   (no_connect (at 41.91 149.225))
+  (no_connect (at 51.435 107.95))
+  (no_connect (at 51.435 110.49))
+  (no_connect (at 51.435 113.03))
+  (no_connect (at 51.435 115.57))
   (no_connect (at 76.2 144.145))
   (no_connect (at 135.255 100.965))
@@
     (stroke (width 0) (type solid) (color 0 0 0 0))
   )
+  (wire (pts (xy 26.035 93.345) (xy 28.575 93.345))
+    (stroke (width 0) (type solid) (color 0 0 0 0))
+  )
+  (wire (pts (xy 26.035 95.885) (xy 28.575 95.885))
+    (stroke (width 0) (type solid) (color 0 0 0 0))
+  )
+  (wire (pts (xy 26.035 98.425) (xy 28.575 98.425))
+    (stroke (width 0) (type solid) (color 0 0 0 0))
+  )
+  (wire (pts (xy 26.035 100.965) (xy 28.575 100.965))
+    (stroke (width 0) (type solid) (color 0 0 0 0))
+  )
   (wire (pts (xy 28.575 41.91) (xy 26.035 41.91))
     (stroke (width 0) (type solid) (color 0 0 0 0))
@@
     (effects (font (size 1.27 1.27)) (justify left bottom))
   )
+  (label "LT_sw" (at 26.035 93.345 180)
+    (effects (font (size 1.27 1.27)) (justify right bottom))
+  )
+  (label "LM_sw" (at 26.035 95.885 180)
+    (effects (font (size 1.27 1.27)) (justify right bottom))
+  )
+  (label "LB_sw" (at 26.035 98.425 180)
+    (effects (font (size 1.27 1.27)) (justify right bottom))
+  )
+  (label "Col_0" (at 26.035 100.965 180)
+    (effects (font (size 1.27 1.27)) (justify right bottom))
+  )
   (label "vsense" (at 26.035 146.685 0)
     (effects (font (size 1.27 1.27)) (justify left bottom))
   )
+  (label "LT_sw" (at 40.005 24.13 0)
+    (effects (font (size 1.27 1.27)) (justify left bottom))
+  )
+  (label "LM_sw" (at 40.005 41.91 0)
+    (effects (font (size 1.27 1.27)) (justify left bottom))
+  )
+  (label "LB_sw" (at 40.005 59.69 0)
+    (effects (font (size 1.27 1.27)) (justify left bottom))
+  )
   (label "Col_5" (at 41.91 136.525 180)
     (effects (font (size 1.27 1.27)) (justify right bottom))
@@
     (effects (font (size 1.27 1.27)) (justify right bottom))
   )
+  (label "RT_sw" (at 52.07 93.345 180)
+    (effects (font (size 1.27 1.27)) (justify right bottom))
+  )
+  (label "RM_sw" (at 52.07 95.885 180)
+    (effects (font (size 1.27 1.27)) (justify right bottom))
+  )
+  (label "RB_sw" (at 52.07 98.425 180)
+    (effects (font (size 1.27 1.27)) (justify right bottom))
+  )
+  (label "Col_9" (at 52.07 100.965 180)
+    (effects (font (size 1.27 1.27)) (justify right bottom))
+  )
   (label "encA" (at 55.88 73.66 180)
     (effects (font (size 1.27 1.27)) (justify right bottom))
@@
     (effects (font (size 1.27 1.27)) (justify right bottom))
   )
+  (label "RT_sw" (at 262.89 24.13 0)
+    (effects (font (size 1.27 1.27)) (justify left bottom))
+  )
+  (label "RM_sw" (at 262.89 41.91 0)
+    (effects (font (size 1.27 1.27)) (justify left bottom))
+  )
+  (label "RB_sw" (at 262.89 59.69 0)
+    (effects (font (size 1.27 1.27)) (justify left bottom))
+  )
   (symbol (lib_id "power:+3V3") (at 35.56 167.005 90) (unit 1)
     (in_bom yes) (on_board yes)
@@
       (effects (font (size 1.27 1.27)) (justify left))
     )
-    (property "Footprint" "Weteor:JST GH 2Pin" (id 2) (at 180.34 121.031 90)
+    (property "Footprint" "Weteor:Molex PicoBlade 2Pin smt tht" (id 2) (at 180.34 121.031 90)
       (effects (font (size 1.27 1.27)) hide)
     )
@@
     (pin "2")
   )
+  (symbol (lib_id "Connector_Generic:Conn_01x04") (at 33.02 110.49 0) (unit 1)
+    (in_bom yes) (on_board yes) (fields_autoplaced)
+    (property "Reference" "J3" (id 0) (at 35.0521 110.8515 0)
+      (effects (font (size 1.27 1.27)) (justify left))
+    )
+    (property "Value" "Conn_01x04" (id 1) (at 35.0521 113.6266 0)
+      (effects (font (size 1.27 1.27)) (justify left))
+    )
+    (property "Footprint" "Connector_PinHeader_1.27mm:PinHeader_1x04_P1.27mm_Vertical" (id 2) (at 33.02 110.49 0)
+      (effects (font (size 1.27 1.27)) hide)
+    )
+    (property "Datasheet" "~" (id 3) (at 33.02 110.49 0)
+      (effects (font (size 1.27 1.27)) hide)
+    )
+    (pin "1")
+    (pin "2")
+    (pin "3")
+    (pin "4")
+  )
+  (symbol (lib_id "Connector_Generic:Conn_01x04") (at 33.655 95.885 0) (unit 1)
+    (in_bom yes) (on_board yes) (fields_autoplaced)
+    (property "Reference" "J4" (id 0) (at 35.6871 96.2465 0)
+      (effects (font (size 1.27 1.27)) (justify left))
+    )
+    (property "Value" "Conn_01x04" (id 1) (at 35.6871 99.0216 0)
+      (effects (font (size 1.27 1.27)) (justify left))
+    )
+    (property "Footprint" "Connector_PinHeader_1.27mm:PinHeader_1x04_P1.27mm_Vertical" (id 2) (at 33.655 95.885 0)
+      (effects (font (size 1.27 1.27)) hide)
+    )
+    (property "Datasheet" "~" (id 3) (at 33.655 95.885 0)
+      (effects (font (size 1.27 1.27)) hide)
+    )
+    (pin "1")
+    (pin "2")
+    (pin "3")
+    (pin "4")
+  )
+  (symbol (lib_id "Connector_Generic:Conn_01x04") (at 56.515 110.49 0) (unit 1)
+    (in_bom yes) (on_board yes) (fields_autoplaced)
+    (property "Reference" "J5" (id 0) (at 58.5471 110.8515 0)
+      (effects (font (size 1.27 1.27)) (justify left))
+    )
+    (property "Value" "Conn_01x04" (id 1) (at 58.5471 113.6266 0)
+      (effects (font (size 1.27 1.27)) (justify left))
+    )
+    (property "Footprint" "Connector_PinHeader_1.27mm:PinHeader_1x04_P1.27mm_Vertical" (id 2) (at 56.515 110.49 0)
+      (effects (font (size 1.27 1.27)) hide)
+    )
+    (property "Datasheet" "~" (id 3) (at 56.515 110.49 0)
+      (effects (font (size 1.27 1.27)) hide)
+    )
+    (pin "1")
+    (pin "2")
+    (pin "3")
+    (pin "4")
+  )
+  (symbol (lib_id "Connector_Generic:Conn_01x04") (at 57.15 95.885 0) (unit 1)
+    (in_bom yes) (on_board yes) (fields_autoplaced)
+    (property "Reference" "J6" (id 0) (at 59.1821 96.2465 0)
+      (effects (font (size 1.27 1.27)) (justify left))
+    )
+    (property "Value" "Conn_01x04" (id 1) (at 59.1821 99.0216 0)
+      (effects (font (size 1.27 1.27)) (justify left))
+    )
+    (property "Footprint" "Connector_PinHeader_1.27mm:PinHeader_1x04_P1.27mm_Vertical" (id 2) (at 57.15 95.885 0)
+      (effects (font (size 1.27 1.27)) hide)
+    )
+    (property "Datasheet" "~" (id 3) (at 57.15 95.885 0)
+      (effects (font (size 1.27 1.27)) hide)
+    )
+    (pin "1")
+    (pin "2")
+    (pin "3")
+    (pin "4")
+  )
   (symbol (lib_id "Connector_Generic:Conn_01x04") (at 156.845 173.99 180) (unit 1)
     (in_bom yes) (on_board yes)
@@
       (effects (font (size 1.27 1.27)) (justify left))
     )
-    (property "Footprint" "Weteor:JST Gh Molex PicoBlade 4Pin" (id 2) (at 156.845 173.99 0)
+    (property "Footprint" "Weteor:Molex PicoBlade 4Pin smt tht" (id 2) (at 156.845 173.99 0)
       (effects (font (size 1.27 1.27)) hide)
     )
@@
     )
     (path "/f3897332-b911-4d20-b857-589fddf122c4"
-      (reference "BT1") (unit 1) (value "Battery_Cell") (footprint "Weteor:JST GH 2Pin")
+      (reference "BT1") (unit 1) (value "Battery_Cell") (footprint "Weteor:Molex PicoBlade 2Pin smt tht")
     )
     (path "/af2ab640-9090-4753-be8a-4692bed2bd46"
@@
     )
     (path "/a6d99b8d-3167-4c55-b34d-7b560562ab80"
-      (reference "J2") (unit 1) (value "BL_CONN") (footprint "Weteor:JST Gh Molex PicoBlade 4Pin")
+      (reference "J2") (unit 1) (value "BL_CONN") (footprint "Weteor:Molex PicoBlade 4Pin smt tht")
+    )
+    (path "/4269e49b-451c-42ef-bd2b-667fbc86b4f8"
+      (reference "J3") (unit 1) (value "Conn_01x04") (footprint "Connector_PinHeader_1.27mm:PinHeader_1x04_P1.27mm_Vertical")
+    )
+    (path "/709e5e29-304b-4f96-a141-345fb3767a24"
+      (reference "J4") (unit 1) (value "Conn_01x04") (footprint "Connector_PinHeader_1.27mm:PinHeader_1x04_P1.27mm_Vertical")
+    )
+    (path "/bb1f28e6-07fd-4b40-b827-c9415be9d20e"
+      (reference "J5") (unit 1) (value "Conn_01x04") (footprint "Connector_PinHeader_1.27mm:PinHeader_1x04_P1.27mm_Vertical")
+    )
+    (path "/d770d2c8-3991-4e2a-9ee3-795a62a0de85"
+      (reference "J6") (unit 1) (value "Conn_01x04") (footprint "Connector_PinHeader_1.27mm:PinHeader_1x04_P1.27mm_Vertical")
     )
     (path "/b6bcf90d-a0e8-4ded-bb15-731310636c04"
