File: pcb/tipper_tf/TipperTF.kicad_sch (KiCad schematic)
At the start: 114 parts, among them J1 USB_C Main, J2 BL_CONN, J3 Conn_01x04, J4 Conn_01x04, J5 Conn_01x04, J6 Conn_01x04, Q1 AO3401A, SW1 SW_Push, SW10 SW_Push, SW11 SW_Push, SW12 SW_Push, SW13 SW_Push, SW14 SW_Push, SW15 SW_Push, SW16 SW_Push, SW17 SW_Push, SW18 SW_Push, SW19 SW_Push, SW2 SW_Push, SW20 SW_Push, SW21 SW_Push, SW22 SW_Push, SW23 SW_Push, SW24 SW_Push, SW25 SW_Push, SW26 SW_Push, SW27 SW_Push, SW28 SW_Push, SW29 SW_Push, SW3 SW_Push, SW30 SW_Push, SW31 SW_Push, SW32 SW_Push, SW33 SW_Push, SW34 SW_Push, SW35 SW_Push, SW36 Rotary_Encoder_Switch, SW37 SW_RESET, SW4 ON_OFF, SW5 SW_Push, SW6 SW_Push, SW7 SW_Push, SW8 SW_Push, SW9 SW_Push, U1 MS88SF2, U2 TP4056, U3 XC6206PxxxMR-Regulator_Linear, U4 DW01A, U5 FS8205, U6 USBLC6-2SC6

Commit message: pcb almost ready
Parts:
- added J7: Conn_01x10, Connector_FFC-FPC:Molex_200528-0100_1x10-1MP_P1.00mm_Horizontal, symbol Connector_Generic:Conn_01x10
Connections:
- net Col_1: now also D1.1 (K), D13.1 (K), D2.1 (K), D3.1 (K), D32.1 (K), D33.1 (K), D34.1 (K), U1.4 (P0.02); no longer SW5.1, SW6.1, SW7.1, U1.21 (P0.20)
- net Col_2: now also D17.1 (K), D29.1 (K), D30.1 (K), D31.1 (K), D4.1 (K), D5.1 (K), D6.1 (K), U1.5 (P0.29); no longer SW10.1, SW36.S1, SW8.1, SW9.1, U1.19 (P0.15)
- net Col_3: now also D21.1 (K), D26.1 (K), D27.1 (K), D28.1 (K), D7.1 (K), D8.1 (K), D9.1 (K), U1.7 (P0.26); no longer SW11.1, SW12.1, SW13.1, SW14.1, U1.18 (P0.13)
- net Col_4: now also D10.1 (K), D11.1 (K), D12.1 (K), D22.1 (K), D23.1 (K), D24.1 (K), D25.1 (K); no longer SW15.1, SW16.1, SW17.1, SW18.1
- net Col_5: now also D14.1 (K), D15.1 (K), D16.1 (K), D18.1 (K), D19.1 (K), D20.1 (K), D35.1 (K), U1.22 (P0.22); no longer SW19.1, SW20.1, SW21.1, SW22.1, U1.2 (P1.13)
- net Row_1: now also J3.1 (Pin_1), SW1.1, SW11.1, SW15.1, SW5.1, SW8.1, U1.18 (P0.13); no longer D11.1 (K), D15.1 (K), D19.1 (K), D2.1 (K), D23.1 (K), D27.1 (K), D30.1 (K), D33.1 (K), D5.1 (K), D8.1 (K), U1.11 (P1.09)
- net Row_2: now also J3.2 (Pin_2), SW12.1, SW16.1, SW2.1, SW6.1, SW9.1, U1.19 (P0.15); no longer D12.1 (K), D16.1 (K), D20.1 (K), D24.1 (K), D28.1 (K), D3.1 (K), D31.1 (K), D34.1 (K), D6.1 (K), D9.1 (K), U1.10 (P0.08)
- net Row_3: now also J3.3 (Pin_3), SW10.1, SW13.1, SW17.1, SW3.1, SW7.1, U1.21 (P0.20); no longer D13.1 (K), D17.1 (K), D21.1 (K), D25.1 (K), D35.1 (K), U1.9 (P0.06)
- net Row_4: now reaches J5.1 (Pin_1)
- net Row_4: now also SW19.1, SW23.1, SW27.1, SW30.1, SW33.1, U1.12 (P0.12)
- net Row_5: now reaches J5.2 (Pin_2)
- net Row_5: now also SW20.1, SW24.1, SW28.1, SW31.1, SW34.1, U1.11 (P1.09)
- net Row_6: now reaches J5.3 (Pin_3)
- net Row_6: now also SW21.1, SW25.1, SW29.1, SW32.1, SW35.1, U1.10 (P0.08)
- net Row_7: now reaches U1.24 (P1.00)
- net Row_7: now also SW14.1, SW18.1, SW22.1, SW26.1, SW36.S1
- removed net Col_0: J4.4 (Pin_4), SW1.1, SW2.1, SW3.1, U1.22 (P0.22)
- removed net Col_6: SW23.1, SW24.1, SW25.1, SW26.1, U1.8 (P0.04)
- removed net Col_7: SW27.1, SW28.1, SW29.1, U1.5 (P0.29)
- removed net Col_8: SW30.1, SW31.1, SW32.1, U1.4 (P0.02)
- removed net Col_9: J6.4 (Pin_4), SW33.1, SW34.1, SW35.1, U1.3 (P1.15)
- removed net Row_0: D1.1 (K), D10.1 (K), D14.1 (K), D18.1 (K), D22.1 (K), D26.1 (K), D29.1 (K), D32.1 (K), D4.1 (K), D7.1 (K), U1.12 (P0.12)
- no-connect marks 15 -> 10
Other:
- moved on the sheet: D1, D10, D11, D12, D13, D14, D15, D16, D17, D18, D19, D2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

Commit message: fix main pcb, new matrix layout, display support, new screwhole positions
Parts:
- J7: footprint Connector_FFC-FPC:Molex_200528-0100_1x10-1MP_P1.00mm_Horizontal -> Connector_FFC-FPC:TE_1-84953-0_1x10-1MP_P1.0mm_Horizontal
Connections:
- net encA is gone; now on net DC_encA: SW36.A, U1.27 (P0.09)
- net encB is gone; now on net CS_encB: SW36.B, U1.28 (P0.10)
- net +3V3: now also J7.10 (Pin_10)
- net GND: now also J7.1 (Pin_1), J7.2 (Pin_2)
- net MOSI: now reaches J7.3 (Pin_3)
- net MOSI: now also U1.8 (P0.04)
- net SCLK: now reaches J7.4 (Pin_4)
- net SCLK: now also U1.9 (P0.06)
- net CS_encB: now reaches J7.5 (Pin_5)
- net DC_encA: now reaches J7.6 (Pin_6)
- net RESET_D: now reaches J7.7 (Pin_7)
- net RESET_D: now also U1.3 (P1.15)
- net BUSY: now reaches J7.8 (Pin_8)
- net BUSY: now also U1.2 (P1.13)
- no-connect marks 10 -> 11
Changed lines of the file:
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@@
   (junction (at 71.12 187.325) (diameter 1.016) (color 0 0 0 0))
   (junction (at 78.74 167.005) (diameter 1.016) (color 0 0 0 0))
+  (junction (at 86.995 76.835) (diameter 0) (color 0 0 0 0))
   (junction (at 87.63 31.75) (diameter 1.016) (color 0 0 0 0))
   (junction (at 87.63 38.1) (diameter 1.016) (color 0 0 0 0))
@@
   (no_connect (at 51.435 115.57))
   (no_connect (at 52.07 100.965))
+  (no_connect (at 88.9 97.155))
   (no_connect (at 135.255 100.965))
   (no_connect (at 217.17 131.445))
@@
     (stroke (width 0) (type solid) (color 0 0 0 0))
   )
+  (wire (pts (xy 84.455 76.835) (xy 86.995 76.835))
+    (stroke (width 0) (type default) (color 0 0 0 0))
+  )
+  (wire (pts (xy 84.455 99.695) (xy 88.9 99.695))
+    (stroke (width 0) (type default) (color 0 0 0 0))
+  )
   (wire (pts (xy 85.725 25.4) (xy 87.63 25.4))
     (stroke (width 0) (type solid) (color 0 0 0 0))
@@
     (stroke (width 0) (type solid) (color 0 0 0 0))
   )
+  (wire (pts (xy 85.725 81.915) (xy 88.9 81.915))
+    (stroke (width 0) (type default) (color 0 0 0 0))
+  )
+  (wire (pts (xy 85.725 84.455) (xy 88.9 84.455))
+    (stroke (width 0) (type default) (color 0 0 0 0))
+  )
+  (wire (pts (xy 85.725 86.995) (xy 88.9 86.995))
+    (stroke (width 0) (type default) (color 0 0 0 0))
+  )
+  (wire (pts (xy 85.725 89.535) (xy 88.9 89.535))
+    (stroke (width 0) (type default) (color 0 0 0 0))
+  )
+  (wire (pts (xy 85.725 92.075) (xy 88.9 92.075))
+    (stroke (width 0) (type default) (color 0 0 0 0))
+  )
+  (wire (pts (xy 85.725 94.615) (xy 88.9 94.615))
+    (stroke (width 0) (type default) (color 0 0 0 0))
+  )
+  (wire (pts (xy 86.995 76.835) (xy 88.9 76.835))
+    (stroke (width 0) (type default) (color 0 0 0 0))
+  )
+  (wire (pts (xy 86.995 79.375) (xy 86.995 76.835))
+    (stroke (width 0) (type default) (color 0 0 0 0))
+  )
   (wire (pts (xy 87.63 25.4) (xy 87.63 31.75))
     (stroke (width 0) (type solid) (color 0 0 0 0))
@@
     (stroke (width 0) (type solid) (color 0 0 0 0))
   )
+  (wire (pts (xy 88.9 79.375) (xy 86.995 79.375))
+    (stroke (width 0) (type default) (color 0 0 0 0))
+  )
   (wire (pts (xy 92.075 27.305) (xy 92.075 25.4))
     (stroke (width 0) (type solid) (color 0 0 0 0))
@@
     (effects (font (size 1.27 1.27)) (justify left bottom))
   )
+  (label "BUSY" (at 41.91 136.525 180)
+    (effects (font (size 1.27 1.27)) (justify right bottom))
+  )
+  (label "RESET_D" (at 41.91 139.065 180)
+    (effects (font (size 1.27 1.27)) (justify right bottom))
+  )
   (label "Col_1" (at 41.91 141.605 180)
     (effects (font (size 1.27 1.27)) (justify right bottom))
@@
     (effects (font (size 1.27 1.27)) (justify right bottom))
   )
+  (label "MOSI" (at 41.91 151.765 180)
+    (effects (font (size 1.27 1.27)) (justify right bottom))
+  )
+  (label "SCLK" (at 41.91 154.305 180)
+    (effects (font (size 1.27 1.27)) (justify right bottom))
+  )
   (label "Row_6" (at 41.91 156.845 180)
     (effects (font (size 1.27 1.27)) (justify right bottom))
@@
     (effects (font (size 1.27 1.27)) (justify right bottom))
   )
-  (label "encB" (at 76.2 133.985 0)
+  (label "CS_encB" (at 76.2 133.985 0)
     (effects (font (size 1.27 1.27)) (justify left bottom))
   )
-  (label "encA" (at 76.2 136.525 0)
+  (label "DC_encA" (at 76.2 136.525 0)
     (effects (font (size 1.27 1.27)) (justify left bottom))
   )
@@
     (effects (font (size 1.27 1.27)) (justify left bottom))
   )
+  (label "MOSI" (at 85.725 81.915 180)
+    (effects (font (size 1.27 1.27)) (justify right bottom))
+  )
+  (label "SCLK" (at 85.725 84.455 180)
+    (effects (font (size 1.27 1.27)) (justify right bottom))
+  )
+  (label "CS_encB" (at 85.725 86.995 180)
+    (effects (font (size 1.27 1.27)) (justify right bottom))
+  )
+  (label "DC_encA" (at 85.725 89.535 180)
+    (effects (font (size 1.27 1.27)) (justify right bottom))
+  )
+  (label "RESET_D" (at 85.725 92.075 180)
+    (effects (font (size 1.27 1.27)) (justify right bottom))
+  )
+  (label "BUSY" (at 85.725 94.615 180)
+    (effects (font (size 1.27 1.27)) (justify right bottom))
+  )
   (label "reset" (at 92.71 154.305 180)
     (effects (font (size 1.27 1.27)) (justify right bottom))
@@
     (effects (font (size 1.27 1.27)) (justify left bottom))
   )
-  (label "encA" (at 130.175 69.85 180)
+  (label "DC_encA" (at 130.175 69.85 180)
     (effects (font (size 1.27 1.27)) (justify right bottom))
   )
-  (label "encB" (at 130.175 74.93 180)
+  (label "CS_encB" (at 130.175 74.93 180)
     (effects (font (size 1.27 1.27)) (justify right bottom))
   )
@@
     (pin "1")
   )
+  (symbol (lib_id "power:+3V3") (at 84.455 99.695 90) (unit 1)
+    (in_bom yes) (on_board yes)
+    (property "Reference" "#PWR0103" (id 0) (at 88.265 99.695 0)
+      (effects (font (size 1.27 1.27)) hide)
+    )
+    (property "Value" "+3V3" (id 1) (at 81.2038 99.314 90)
+      (effects (font (size 1.27 1.27)) (justify left))
+    )
+    (property "Footprint" "" (id 2) (at 84.455 99.695 0)
+      (effects (font (size 1.27 1.27)) hide)
+    )
+    (property "Datasheet" "" (id 3) (at 84.455 99.695 0)
+      (effects (font (size 1.27 1.27)) hide)
+    )
+    (pin "1")
+  )
   (symbol (lib_id "power:+3V3") (at 168.275 194.31 270) (unit 1)
     (in_bom yes) (on_board yes)
@@
     (pin "1")
   )
+  (symbol (lib_id "power:GND") (at 84.455 76.835 270) (unit 1)
+    (in_bom yes) (on_board yes)
+    (property "Reference" "#PWR0102" (id 0) (at 78.105 76.835 0)
+      (effects (font (size 1.27 1.27)) hide)
+    )
+    (property "Value" "GND" (id 1) (at 80.0608 76.962 0))
+    (property "Footprint" "" (id 2) (at 84.455 76.835 0)
+      (effects (font (size 1.27 1.27)) hide)
+    )
+    (property "Datasheet" "" (id 3) (at 84.455 76.835 0)
+      (effects (font (size 1.27 1.27)) hide)
+    )
+    (pin "1")
+  )
   (symbol (lib_id "power:GND") (at 96.52 177.165 0) (unit 1)
     (in_bom yes) (on_board yes)
@@
       (effects (font (size 1.27 1.27)) (justify left))
     )
-    (property "Footprint" "Connector_FFC-FPC:Molex_200528-0100_1x10-1MP_P1.00mm_Horizontal" (id 2) (at 93.98 86.995 0)
+    (property "Footprint" "Connector_FFC-FPC:TE_1-84953-0_1x10-1MP_P1.0mm_Horizontal" (id 2) (at 93.98 86.995 0)
       (effects (font (size 1.27 1.27)) hide)
     )
@@
       (reference "#PWR0101") (unit 1) (value "+3V3") (footprint "")
     )
+    (path "/5b32c50c-af45-41d6-981f-c9c7c19a818c"
+      (reference "#PWR0102") (unit 1) (value "GND") (footprint "")
+    )
+    (path "/43ce501c-3e99-4d41-be5a-2df646f70482"
+      (reference "#PWR0103") (unit 1) (value "+3V3") (footprint "")
+    )
     (path "/f3897332-b911-4d20-b857-589fddf122c4"
       (reference "BT1") (unit 1) (value "Battery_Cell") (footprint "Weteor:Molex PicoBlade 2Pin smt tht")
@@
     )
     (path "/03a53f72-d661-4af4-80cd-1ce702c05b16"
-      (reference "J7") (unit 1) (value "Conn_01x10") (footprint "Connector_FFC-FPC:Molex_200528-0100_1x10-1MP_P1.00mm_Horizontal")
+      (reference "J7") (unit 1) (value "Conn_01x10") (footprint "Connector_FFC-FPC:TE_1-84953-0_1x10-1MP_P1.0mm_Horizontal")
     )
     (path "/b6bcf90d-a0e8-4ded-bb15-731310636c04"

Commit message: pcb update rev2 prod.
Parts:
- removed D35: D, Weteor:D_SOD-123, symbol Device:D_Small
- removed SW36: Rotary_Encoder_Switch, Weteor:RotEncoderE11_SMD, symbol Device:Rotary_Encoder_Switch
- BT1: footprint Weteor:Molex PicoBlade 2Pin smt tht -> Connector_PinHeader_2.54mm:PinHeader_1x02_P2.54mm_Vertical
- J2: footprint Weteor:Molex PicoBlade 4Pin smt tht -> Connector_PinHeader_2.54mm:PinHeader_1x04_P2.54mm_Vertical
- J7: footprint Connector_FFC-FPC:TE_1-84953-0_1x10-1MP_P1.0mm_Horizontal -> Weteor:FCC 1x10 - JUSHUO AFC01-S10FCA-00
- SW4: footprint Weteor:switch_MSK-12C02_smd -> Weteor:K3-2380S-E1 On-on
Connections:
- net BUSY: now also U1.3 (P1.15); no longer U1.2 (P1.13)
- net MOSI: now also U1.28 (P0.10); no longer U1.8 (P0.04)
- net RESET_D: now also U1.2 (P1.13); no longer U1.3 (P1.15)
- net SCLK: now also U1.27 (P0.09); no longer U1.9 (P0.06)
- net CS_encB renamed CS
- net CS: now also U1.8 (P0.04); no longer U1.28 (P0.10)
- net DC_encA renamed DC
- net DC: now also U1.9 (P0.06); no longer U1.27 (P0.09)
- no-connect marks 11 -> 10
Changed lines of the file:
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@@
   (no_connect (at 26.035 100.965))
   (no_connect (at 27.94 115.57))
-  (no_connect (at 37.465 130.175))
   (no_connect (at 51.435 115.57))
   (no_connect (at 52.07 100.965))
@@
     (stroke (width 0) (type solid) (color 0 0 0 0))
   )
-  (wire (pts (xy 132.08 69.85) (xy 130.175 69.85))
-    (stroke (width 0) (type solid) (color 0 0 0 0))
-  )
-  (wire (pts (xy 132.08 72.39) (xy 124.46 72.39))
-    (stroke (width 0) (type solid) (color 0 0 0 0))
-  )
-  (wire (pts (xy 132.08 74.93) (xy 130.175 74.93))
-    (stroke (width 0) (type solid) (color 0 0 0 0))
-  )
   (wire (pts (xy 132.715 103.505) (xy 135.255 103.505))
     (stroke (width 0) (type solid) (color 0 0 0 0))
@@
     (stroke (width 0) (type solid) (color 0 0 0 0))
   )
-  (wire (pts (xy 147.32 69.85) (xy 155.575 69.85))
-    (stroke (width 0) (type solid) (color 0 0 0 0))
-  )
-  (wire (pts (xy 147.32 74.93) (xy 149.225 74.93))
-    (stroke (width 0) (type solid) (color 0 0 0 0))
-  )
-  (wire (pts (xy 154.305 74.93) (xy 155.575 74.93))
-    (stroke (width 0) (type solid) (color 0 0 0 0))
-  )
   (wire (pts (xy 156.21 25.4) (xy 156.845 25.4))
     (stroke (width 0) (type solid) (color 0 0 0 0))
@@
     (effects (font (size 1.27 1.27)) (justify left bottom))
   )
-  (label "BUSY" (at 41.91 136.525 180)
+  (label "RESET_D" (at 41.91 136.525 180)
     (effects (font (size 1.27 1.27)) (justify right bottom))
   )
-  (label "RESET_D" (at 41.91 139.065 180)
+  (label "BUSY" (at 41.91 139.065 180)
     (effects (font (size 1.27 1.27)) (justify right bottom))
   )
@@
     (effects (font (size 1.27 1.27)) (justify right bottom))
   )
-  (label "MOSI" (at 41.91 151.765 180)
+  (label "CS" (at 41.91 151.765 180)
     (effects (font (size 1.27 1.27)) (justify right bottom))
   )
-  (label "SCLK" (at 41.91 154.305 180)
+  (label "DC" (at 41.91 154.305 180)
     (effects (font (size 1.27 1.27)) (justify right bottom))
   )
@@
     (effects (font (size 1.27 1.27)) (justify right bottom))
   )
-  (label "CS_encB" (at 76.2 133.985 0)
+  (label "MOSI" (at 76.2 133.985 0)
     (effects (font (size 1.27 1.27)) (justify left bottom))
   )
-  (label "DC_encA" (at 76.2 136.525 0)
+  (label "SCLK" (at 76.2 136.525 0)
     (effects (font (size 1.27 1.27)) (justify left bottom))
   )
@@
     (effects (font (size 1.27 1.27)) (justify right bottom))
   )
-  (label "CS_encB" (at 85.725 86.995 180)
+  (label "CS" (at 85.725 86.995 180)
     (effects (font (size 1.27 1.27)) (justify right bottom))
   )
-  (label "DC_encA" (at 85.725 89.535 180)
+  (label "DC" (at 85.725 89.535 180)
     (effects (font (size 1.27 1.27)) (justify right bottom))
   )
@@
     (effects (font (size 1.27 1.27)) (justify left bottom))
   )
-  (label "DC_encA" (at 130.175 69.85 180)
-    (effects (font (size 1.27 1.27)) (justify right bottom))
-  )
-  (label "CS_encB" (at 130.175 74.93 180)
-    (effects (font (size 1.27 1.27)) (justify right bottom))
-  )
   (label "vbus" (at 130.81 95.885 0)
     (effects (font (size 1.27 1.27)) (justify left bottom))
@@
     (effects (font (size 1.27 1.27)) (justify left bottom))
   )
-  (label "Row_7" (at 155.575 69.85 0)
-    (effects (font (size 1.27 1.27)) (justify left bottom))
-  )
-  (label "Col_5" (at 155.575 74.93 0)
-    (effects (font (size 1.27 1.27)) (justify left bottom))
-  )
   (label "swclk" (at 165.1 168.91 0)
     (effects (font (size 1.27 1.27)) (justify left bottom))
@@
     (pin "1")
   )
-  (symbol (lib_id "power:GND") (at 124.46 72.39 270) (unit 1)
-    (in_bom yes) (on_board yes)
-    (property "Reference" "#PWR018" (id 0) (at 118.11 72.39 0)
-      (effects (font (size 1.27 1.27)) hide)
-    )
-    (property "Value" "GND" (id 1) (at 121.2088 72.517 90)
-      (effects (font (size 1.27 1.27)) (justify right))
-    )
-    (property "Footprint" "" (id 2) (at 124.46 72.39 0)
-      (effects (font (size 1.27 1.27)) hide)
-    )
-    (property "Datasheet" "" (id 3) (at 124.46 72.39 0)
-      (effects (font (size 1.27 1.27)) hide)
-    )
-    (pin "1")
-  )
   (symbol (lib_id "power:GND") (at 147.955 112.395 0) (unit 1)
     (in_bom yes) (on_board yes)
@@
     (pin "2")
   )
-  (symbol (lib_id "Device:D_Small") (at 151.765 74.93 180) (unit 1)
-    (in_bom yes) (on_board yes)
-    (property "Reference" "D35" (id 0) (at 150.5966 73.152 90)
-      (effects (font (size 1.27 1.27)) (justify right))
-    )
-    (property "Value" "D" (id 1) (at 152.908 73.152 90)
-      (effects (font (size 1.27 1.27)) (justify right))
-    )
-    (property "Footprint" "Weteor:D_SOD-123" (id 2) (at 151.765 74.93 90)
-      (effects (font (size 1.27 1.27)) hide)
-    )
-    (property "Datasheet" "~" (id 3) (at 151.765 74.93 90)
-      (effects (font (size 1.27 1.27)) hide)
-    )
-    (pin "1")
-    (pin "2")
-  )
   (symbol (lib_id "Device:D_Small") (at 159.385 25.4 180) (unit 1)
     (in_bom yes) (on_board yes)
@@
       (effects (font (size 1.27 1.27)) (justify left))
     )
-    (property "Footprint" "Weteor:Molex PicoBlade 2Pin smt tht" (id 2) (at 180.34 121.031 90)
+    (property "Footprint" "Connector_PinHeader_2.54mm:PinHeader_1x02_P2.54mm_Vertical" (id 2) (at 180.34 121.031 90)
       (effects (font (size 1.27 1.27)) hide)
     )
@@
       (effects (font (size 1.27 1.27)) (justify left))
     )
-    (property "Footprint" "Weteor:Molex PicoBlade 4Pin smt tht" (id 2) (at 156.845 173.99 0)
+    (property "Footprint" "Connector_PinHeader_2.54mm:PinHeader_1x04_P2.54mm_Vertical" (id 2) (at 156.845 173.99 0)
       (effects (font (size 1.27 1.27)) hide)
     )
@@
     (property "Reference" "SW4" (id 0) (at 58.42 172.9232 0))
     (property "Value" "ON_OFF" (id 1) (at 58.42 175.2346 0))
-    (property "Footprint" "Weteor:switch_MSK-12C02_smd" (id 2) (at 58.42 179.705 0)
+    (property "Footprint" "Weteor:K3-2380S-E1 On-on" (id 2) (at 58.42 179.705 0)
       (effects (font (size 1.27 1.27)) hide)
     )
@@
     (pin "3")
   )
-  (symbol (lib_id "Device:Rotary_Encoder_Switch") (at 139.7 72.39 0) (unit 1)
-    (in_bom yes) (on_board yes)
-    (property "Reference" "SW36" (id 0) (at 139.7 63.0682 0))
-    (property "Value" "Rotary_Encoder_Switch" (id 1) (at 139.7 65.3796 0))
-    (property "Footprint" "Weteor:RotEncoderE11_SMD" (id 2) (at 135.89 68.326 0)
-      (effects (font (size 1.27 1.27)) hide)
-    )
-    (property "Datasheet" "~" (id 3) (at 139.7 65.786 0)
-      (effects (font (size 1.27 1.27)) hide)
-    )
-    (pin "A")
-    (pin "B")
-    (pin "C")
-    (pin "S1")
-    (pin "S2")
-  )
   (symbol (lib_id "Connector_Generic:Conn_01x10") (at 93.98 86.995 0) (unit 1)
     (in_bom yes) (on_board yes) (fields_autoplaced)
@@
       (effects (font (size 1.27 1.27)) (justify left))
     )
-    (property "Footprint" "Connector_FFC-FPC:TE_1-84953-0_1x10-1MP_P1.0mm_Horizontal" (id 2) (at 93.98 86.995 0)
+    (property "Footprint" "Weteor:FCC 1x10 - JUSHUO AFC01-S10FCA-00" (id 2) (at 93.98 86.995 0)
       (effects (font (size 1.27 1.27)) hide)
     )
@@
       (reference "#PWR017") (unit 1) (value "GND") (footprint "")
     )
-    (path "/00000000-0000-0000-0000-0000613da164"
-      (reference "#PWR018") (unit 1) (value "GND") (footprint "")
-    )
     (path "/e561018b-073b-4aa9-8dd7-eaa3442e083d"
       (reference "#PWR020") (unit 1) (value "GND") (footprint "")
@@
     )
     (path "/f3897332-b911-4d20-b857-589fddf122c4"
-      (reference "BT1") (unit 1) (value "Battery_Cell") (footprint "Weteor:Molex PicoBlade 2Pin smt tht")
+      (reference "BT1") (unit 1) (value "Battery_Cell") (footprint "Connector_PinHeader_2.54mm:PinHeader_1x02_P2.54mm_Vertical")
     )
     (path "/af2ab640-9090-4753-be8a-4692bed2bd46"
@@
       (reference "D34") (unit 1) (value "D") (footprint "Weteor:D_SOD-123")
     )
-    (path "/00000000-0000-0000-0000-000061367980"
-      (reference "D35") (unit 1) (value "D") (footprint "Weteor:D_SOD-123")
-    )
     (path "/eed37b7c-2fb4-4a54-9aa3-bd0f62a07b1e"
       (reference "D36") (unit 1) (value "D_Schottky_Small") (footprint "Diode_SMD:D_SOD-323_HandSoldering")
@@
     )
     (path "/a6d99b8d-3167-4c55-b34d-7b560562ab80"
-      (reference "J2") (unit 1) (value "BL_CONN") (footprint "Weteor:Molex PicoBlade 4Pin smt tht")
+      (reference "J2") (unit 1) (value "BL_CONN") (footprint "Connector_PinHeader_2.54mm:PinHeader_1x04_P2.54mm_Vertical")
     )
     (path "/4269e49b-451c-42ef-bd2b-667fbc86b4f8"
@@
     )
     (path "/03a53f72-d661-4af4-80cd-1ce702c05b16"
-      (reference "J7") (unit 1) (value "Conn_01x10") (footprint "Connector_FFC-FPC:TE_1-84953-0_1x10-1MP_P1.0mm_Horizontal")
+      (reference "J7") (unit 1) (value "Conn_01x10") (footprint "Weteor:FCC 1x10 - JUSHUO AFC01-S10FCA-00")
     )
     (path "/b6bcf90d-a0e8-4ded-bb15-731310636c04"
@@
     )
     (path "/3740da8d-213a-4657-adef-5b388dac4fa7"
-      (reference "SW4") (unit 1) (value "ON_OFF") (footprint "Weteor:switch_MSK-12C02_smd")
+      (reference "SW4") (unit 1) (value "ON_OFF") (footprint "Weteor:K3-2380S-E1 On-on")
     )
     (path "/00000000-0000-0000-0000-000060541030"
@@
       (reference "SW35") (unit 1) (value "SW_Push") (footprint "Weteor:Kailh_Choc_1u")
     )
-    (path "/00000000-0000-0000-0000-0000612b2212"
-      (reference "SW36") (unit 1) (value "Rotary_Encoder_Switch") (footprint "Weteor:RotEncoderE11_SMD")
-    )
     (path "/7ee0d235-fae2-459b-92f0-c4c8d65361e5"
