File: pcb/tipper_tf/TipperTF.kicad_pcb (KiCad board)
At the start: 2 copper layers, 229.6 x 104.4 mm, 121 parts, among them J1 USB_C Main, J2 BL_CONN, J3 Conn_01x04, J4 Conn_01x04, J5 Conn_01x04, J6 Conn_01x04, J7 Conn_01x10, Q1 AO3401A, SW1 SW_Push, SW10 SW_Push, SW11 SW_Push, SW12 SW_Push, SW13 SW_Push, SW14 SW_Push, SW15 SW_Push, SW16 SW_Push, SW17 SW_Push, SW18 SW_Push, SW19 SW_Push, SW2 SW_Push, SW20 SW_Push, SW21 SW_Push, SW22 SW_Push, SW23 SW_Push, SW24 SW_Push, SW25 SW_Push, SW26 SW_Push, SW27 SW_Push, SW28 SW_Push, SW29 SW_Push, SW3 SW_Push, SW30 SW_Push, SW31 SW_Push, SW32 SW_Push, SW33 SW_Push, SW34 SW_Push, SW35 SW_Push, SW37 SW_RESET, SW4 ON_OFF, SW5 SW_Push, SW6 SW_Push, SW7 SW_Push, SW8 SW_Push, SW9 SW_Push, U1 MS88SF2, U2 TP4056, U3 XC6206PxxxMR-Regulator_Linear, U4 DW01A, U5 FS8205, U6 USBLC6-2SC6

Commit message: new, hopefully corrected version of displayboard
Parts:
- SW1, SW10, SW11, SW12, SW13, SW15, SW16, SW17, SW18, SW19, SW2, SW20, SW21, SW22, SW23, SW24, SW25, SW27, SW28, SW29, SW3, SW30, SW31, SW32, SW33, SW34, SW35, SW5, SW6, SW7, SW8, SW9: footprint Weteor:Kailh_Choc_1u -> Weteor:Kailh_Choc_1u_cutout
- SW14, SW26: footprint Weteor:Kailh_Choc_1.5u -> Weteor:Kailh_Choc_1.5u_cutout

Commit message: newest revision of pcb, adds support for choc V2 (WITH CHOC SPACING) and tighening the holes for V1
Parts:
- SW1, SW10, SW11, SW12, SW13, SW15, SW16, SW17, SW18, SW19, SW2, SW20, SW21, SW22, SW23, SW24, SW25, SW27, SW28, SW29, SW3, SW30, SW31, SW32, SW33, SW34, SW35, SW5, SW6, SW7, SW8, SW9: footprint Weteor:Kailh_Choc_1u_cutout -> Weteor:Kailh_Choc1_2_1u_1.7Hole
- SW14, SW26: footprint Weteor:Kailh_Choc_1.5u_cutout -> Weteor:Kailh_Choc1_2_1.5u_1.7Hole
- moved D21 9.70 mm to (136.6, 158.3)
- moved C10 9.09 mm to (137.2, 98.1)
- moved R15 8.86 mm to (137.3, 94.2)
- moved D23 8.34 mm to (166.8, 99.1)
- moved SW23 8.34 mm to (162.2, 87.6)
- moved SW4 8.34 mm to (111.1, 80.2)
- moved D1 8.34 mm to (23.2, 76.6)
- moved D27 8.34 mm to (182.1, 89.0)
- moved J2 8.34 mm to (94.6, 145.5)
- moved SW33 8.34 mm to (225.4, 81.2)
- moved D29 8.34 mm to (197.6, 71.3)
- moved SW20 8.34 mm to (151.5, 109.9)
- moved J7 8.34 mm to (53.3, 135.6)
- moved SW35 8.34 mm to (228.7, 115.1)
- moved D37 8.34 mm to (137.1, 80.0)
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Routing:
- net /vbat: track 131.7 -> 121.6 mm, vias 6 -> 4
- net /vsense: track 8.21 -> 13.7 mm
- net /Col_4: track 234.8 -> 238.3 mm
- net /RB_sw: track 43.7 -> 40.6 mm
- net /Col_5: track 190.1 -> 192.9 mm
- net /Col_3: track 281.0 -> 283.6 mm
- net /Row_7: track 114.7 -> 117.2 mm
- net /Col_1: track 339.9 -> 337.4 mm
- net Net-(C2-Pad1): track 106.3 -> 108.6 mm
- net /Col_2: track 309.0 -> 311.2 mm
- net Net-(D17-Pad2): track 13.6 -> 15.7 mm
- net /swdio: track 27.2 -> 28.6 mm
- net /Row_6: track 145.9 -> 144.6 mm
- net +3V3: track 172.0 -> 171.0 mm
- net /RM_sw: track 18.2 -> 19.2 mm
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Other:
- board text added: "(c)weteor :: V2.1-20220107 :: github.com/weteor/Tipper-TF :: CERN-OHL-P v2"
