File: pcb/DisplayDaughterboardEPD/DisplayDaughterboardEPD.kicad_sch (KiCad schematic)
At the start: 23 parts, among them J1 Conn_01x10_Female, J2 Conn_01x24_Female, Q1 SI1308

Commit message: daughterboard update for prod rev2
Parts:
- J1: footprint Connector_FFC-FPC:TE_1-84953-0_1x10-1MP_P1.0mm_Horizontal -> weteor:FCC 1x10 - JUSHUO AFC01-S10FCA-00
Changed lines of the file:
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@@
       (effects (font (size 1.27 1.27)) (justify left))
     )
-    (property "Footprint" "Connector_FFC-FPC:TE_1-84953-0_1x10-1MP_P1.0mm_Horizontal" (id 2) (at 57.15 69.85 0)
+    (property "Footprint" "weteor:FCC 1x10 - JUSHUO AFC01-S10FCA-00" (id 2) (at 57.15 69.85 0)
       (effects (font (size 1.27 1.27)) hide)
     )
@@
     )
     (path "/d451443c-71bc-4eb0-921c-3e7d2582980c"
-      (reference "J1") (unit 1) (value "Conn_01x10_Female") (footprint "Connector_FFC-FPC:TE_1-84953-0_1x10-1MP_P1.0mm_Horizontal")
+      (reference "J1") (unit 1) (value "Conn_01x10_Female") (footprint "weteor:FCC 1x10 - JUSHUO AFC01-S10FCA-00")
     )
     (path "/456287bd-7bae-409b-8ff0-e0544aef55e9"

Commit message: new, hopefully corrected version of displayboard
Parts:
- removed Q1: SI1308, Package_TO_SOT_SMD:SOT-323_SC-70, symbol weteor:SI1308
- added Q1: AO3400A, Package_TO_SOT_SMD:SOT-23, symbol Transistor_FET:AO3400A
- L1: footprint Inductor_SMD:L_0603_1608Metric -> Inductor_SMD:L_1210_3225Metric
- R1: value 2.2R -> 0.47R
Connections:
- net RESE: now also Q1.2 (S)
- net at C3.2, D3.2 (A), L1.2: now also Q1.3 (D)
- net at J2.23 (Pin_23), R2.2: now also Q1.1 (G)
Changed lines of the file:
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@@
     (property "Reference" "L1" (id 0) (at 138.43 75.0274 90))
     (property "Value" "10uH" (id 1) (at 138.43 77.8025 90))
-    (property "Footprint" "Inductor_SMD:L_0603_1608Metric" (id 2) (at 138.43 79.375 0)
+    (property "Footprint" "Inductor_SMD:L_1210_3225Metric" (id 2) (at 138.43 79.375 0)
       (effects (font (size 1.27 1.27)) hide)
     )
@@
       (effects (font (size 1.27 1.27)) (justify left))
     )
-    (property "Value" "2.2R" (id 1) (at 136.1187 54.5716 0)
+    (property "Value" "0.47R" (id 1) (at 136.1187 54.5716 0)
       (effects (font (size 1.27 1.27)) (justify left))
     )
@@
     (pin "2")
   )
-  (symbol (lib_id "weteor:SI1308") (at 148.59 55.245 180) (unit 1)
-    (in_bom yes) (on_board yes) (fields_autoplaced)
-    (property "Reference" "Q1" (id 0) (at 144.6529 54.3365 0)
-      (effects (font (size 1.27 1.27)) (justify left))
-    )
-    (property "Value" "SI1308" (id 1) (at 144.6529 57.1116 0)
-      (effects (font (size 1.27 1.27)) (justify left))
-    )
-    (property "Footprint" "Package_TO_SOT_SMD:SOT-323_SC-70" (id 2) (at 147.32 55.245 0)
-      (effects (font (size 1.27 1.27)) hide)
-    )
-    (property "Datasheet" "" (id 3) (at 147.32 55.245 0)
-      (effects (font (size 1.27 1.27)) hide)
+  (symbol (lib_id "Transistor_FET:AO3400A") (at 149.86 55.245 180) (unit 1)
+    (in_bom yes) (on_board yes) (fields_autoplaced)
+    (property "Reference" "Q1" (id 0) (at 144.653 54.3365 0)
+      (effects (font (size 1.27 1.27)) (justify left))
+    )
+    (property "Value" "AO3400A" (id 1) (at 144.653 57.1116 0)
+      (effects (font (size 1.27 1.27)) (justify left))
+    )
+    (property "Footprint" "Package_TO_SOT_SMD:SOT-23" (id 2) (at 144.78 53.34 0)
+      (effects (font (size 1.27 1.27) italic) (justify left) hide)
+    )
+    (property "Datasheet" "http://www.aosmd.com/pdfs/datasheet/AO3400A.pdf" (id 3) (at 149.86 55.245 0)
+      (effects (font (size 1.27 1.27)) (justify left) hide)
     )
     (pin "1")
@@
     )
     (path "/68d13201-115a-4f18-baf2-4bf3002dbb6b"
-      (reference "L1") (unit 1) (value "10uH") (footprint "Inductor_SMD:L_0603_1608Metric")
-    )
-    (path "/a49f4a63-6a0c-44c3-bb00-24a6bd7cf5cb"
-      (reference "Q1") (unit 1) (value "SI1308") (footprint "Package_TO_SOT_SMD:SOT-323_SC-70")
+      (reference "L1") (unit 1) (value "10uH") (footprint "Inductor_SMD:L_1210_3225Metric")
+    )
+    (path "/7482d2d6-f574-45a3-b28f-81ddf40a6a18"
+      (reference "Q1") (unit 1) (value "AO3400A") (footprint "Package_TO_SOT_SMD:SOT-23")
     )
     (path "/900ec7a9-6e30-49e1-af17-082573c1771c"
-      (reference "R1") (unit 1) (value "2.2R") (footprint "Resistor_SMD:R_0603_1608Metric")
+      (reference "R1") (unit 1) (value "0.47R") (footprint "Resistor_SMD:R_0603_1608Metric")
     )
     (path "/fed19b1b-ee3a-46e5-8b29-15f6518d369f"
